File: Odb225JKK_TEST4.kicad_pcb (KiCad board)
At the start: 2 copper layers, 100 x 40 mm, 117 parts, among them IC4 DSPIC33FJ128MC804-PT, J1 I2C, J2 USB4110-GF-A, J3 PPS, J4 SSB, J5 ANT0, J6 ANT0, J7 NMEA, J8 DIAG, J9 ANT0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

Commit message: edit readme
Parts:
- removed C28: 4u7, Capacitor_SMD:C_0603_1608Metric_Pad1.08x0.95mm_HandSolder
- J4: value SSB -> Conn_01x04; footprint Connector_PinHeader_2.54mm:PinHeader_1x02_P2.54mm_Vertical -> Connector_PinHeader_2.54mm:PinHeader_1x04_P2.54mm_Vertical
- R1, R13, R6, R7, R8: value 620R -> 470R
- R19: value 18k -> 470R
- moved J4 2.53 mm to (213.9, 98.5)
Connections:
- net Net-(IC4-PWM1H2/DAC1RP/RP12/CN14/PMD0/RB12) renamed /DIAG-OUT
- R19 pad 1: Net-(C28-Pad1) -> /MOD_IN
- R26 pad 2: Net-(U$1B-OUT) -> /1KHZ
- TP6 pad 1: Net-(U$1B-OUT) -> /1KHZ
- U$1 pad 7: Net-(U$1B-OUT) -> /1KHZ
Routing:
- net /1KHZ: track 0.00 -> 20.2 mm
- net /MOD_IN: track 98.5 -> 108.0 mm, vias 3 -> 4
- net Net-(J4-Pin_1): track 26.3 -> 34.3 mm
- net Net-(U$1B-OUT): track 5.78 -> 0.00 mm
- net Net-(C28-Pad1): track 3.81 -> 0.00 mm
- net /AUDIO_1KHZ: track 30.9 -> 29.3 mm
- net GND: vias 124 -> 126
Other:
- board text added: "1KHZ"
