File: Odb225JKK_TEST4.kicad_sch (KiCad schematic)
At the start: 112 parts, among them IC4 DSPIC33FJ128MC804-PT, J1 I2C, J2 USB4110-GF-A, J3 PPS, J4 SSB, J5 ANT0, J6 ANT0, J7 NMEA, J8 DIAG, J9 ANT0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

Commit message: edit readme
Parts:
- removed J4: SSB, Connector_PinHeader_2.54mm:PinHeader_1x02_P2.54mm_Vertical, symbol Connector_Generic:Conn_01x02
- added J4: Conn_01x04, Connector_PinHeader_2.54mm:PinHeader_1x04_P2.54mm_Vertical, symbol Connector_Generic:Conn_01x04
- R1, R13, R6, R7, R8: value 620R -> 470R
- R19: value 5k1 -> 470R
Connections:
- net GND: now also J4.2 (Pin_2), J4.3 (Pin_3)
- net 1KHZ: now reaches R26.2, TP6.1, U$1.7 (OUT)
- net 1KHZ: now also J4.4 (Pin_4)
- net at C21.2: now also J4.1 (Pin_1)
Changed lines of the file:
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@@
 	)
 	(junction
+		(at 227.33 116.84)
+		(diameter 0)
+		(color 0 0 0 0)
+	)
+	(junction
 		(at 207.01 220.98)
 		(diameter 0)
@@
 	(wire
 		(pts
+			(xy 227.33 116.84) (xy 236.22 116.84)
+		)
+		(stroke
+			(width 0)
+			(type default)
+		)
+	)
+	(wire
+		(pts
 			(xy 25.4 134.62) (xy 25.4 168.91)
 		)
@@
 	(wire
 		(pts
-			(xy 250.825 114.3) (xy 236.22 114.3)
-		)
-		(stroke
-			(width 0)
-			(type default)
-		)
-	)
-	(wire
-		(pts
 			(xy 240.665 142.24) (xy 240.665 139.065)
 		)
@@
 	(wire
 		(pts
+			(xy 227.33 116.84) (xy 227.33 119.38)
+		)
+		(stroke
+			(width 0)
+			(type default)
+		)
+	)
+	(wire
+		(pts
 			(xy 34.29 219.71) (xy 41.91 219.71)
 		)
@@
 	(wire
 		(pts
+			(xy 227.33 114.3) (xy 250.825 114.3)
+		)
+		(stroke
+			(width 0)
+			(type default)
+		)
+	)
+	(wire
+		(pts
 			(xy 173.99 119.38) (xy 173.99 125.73)
 		)
@@
 	(wire
 		(pts
+			(xy 227.33 121.92) (xy 233.68 121.92)
+		)
+		(stroke
+			(width 0)
+			(type default)
+		)
+	)
+	(wire
+		(pts
 			(xy 355.6 143.51) (xy 355.6 144.78)
 		)
@@
 		)
 	)
+	(label "1KHZ"
+		(at 119.38 241.3 0)
+		(fields_autoplaced yes)
+		(effects
+			(font
+				(size 1.27 1.27)
+			)
+			(justify left bottom)
+		)
+	)
 	(label "MCLR"
 		(at 31.75 152.4 180)
@@
 		)
 	)
+	(label "1KHZ"
+		(at 228.6 121.92 0)
+		(fields_autoplaced yes)
+		(effects
+			(font
+				(size 1.27 1.27)
+			)
+			(justify left bottom)
+		)
+	)
 	(label "LED3"
 		(at 39.37 59.69 90)
@@
 	)
 	(symbol
+		(lib_id "Connector_Generic:Conn_01x04")
+		(at 222.25 116.84 0)
+		(mirror y)
+		(unit 1)
+		(exclude_from_sim no)
+		(in_bom yes)
+		(on_board yes)
+		(dnp no)
+		(fields_autoplaced yes)
+		(property "Reference" "J4"
+			(at 222.25 107.95 0)
+			(effects
+				(font
+					(size 1.27 1.27)
+				)
+			)
+		)
+		(property "Value" "Conn_01x04"
+			(at 222.25 110.49 0)
+			(effects
+				(font
+					(size 1.27 1.27)
+				)
+			)
+		)
+		(property "Footprint" "Connector_PinHeader_2.54mm:PinHeader_1x04_P2.54mm_Vertical"
+			(at 222.25 116.84 0)
+			(effects
+				(font
+					(size 1.27 1.27)
+				)
+				(hide yes)
+			)
+		)
+		(property "Datasheet" "~"
+			(at 222.25 116.84 0)
+			(effects
+				(font
+					(size 1.27 1.27)
+				)
+				(hide yes)
+			)
+		)
+		(property "Description" "Generic connector, single row, 01x04, script generated (kicad-library-utils/schlib/autogen/connector/)"
+			(at 222.25 116.84 0)
+			(effects
+				(font
+					(size 1.27 1.27)
+				)
+				(hide yes)
+			)
+		)
+		(pin "4"
+		)
+		(pin "3"
+		)
+		(pin "1"
+		)
+		(pin "2"
+		)
+		(instances
+			(project "Odb225JKK_TEST4"
+				(path "/fd24851e-81c8-49e1-a423-2c617f6dbaa3"
+					(reference "J4")
+					(unit 1)
+				)
+			)
+		)
+	)
+	(symbol
 		(lib_id "odb225:LEDCHIPLED_0805")
 		(at 39.37 74.93 0)
@@
 			)
 		)
-		(property "Value" "620R"
+		(property "Value" "470R"
 			(at 36.068 63.5 0)
 			(effects
@@
 			)
 		)
-		(property "Value" "620R"
+		(property "Value" "470R"
 			(at 28.448 63.5 0)
 			(effects
@@
 			)
 		)
-		(property "Value" "620R"
+		(property "Value" "470R"
 			(at 20.828 63.5 0)
 			(effects
@@
 			)
 		)
-		(property "Value" "5k1"
+		(property "Value" "470R"
 			(at 71.12 233.172 0)
 			(effects
@@
 			)
 		)
-		(property "Value" "620R"
+		(property "Value" "470R"
 			(at 43.688 63.5 0)
 			(effects
@@
 			)
 		)
-		(property "Value" "620R"
+		(property "Value" "470R"
 			(at 13.208 63.5 0)
 			(effects
@@
 					(unit 1)
 				)
-			)
-		)
-	)
-	(symbol
-		(lib_id "Connector_Generic:Conn_01x02")
-		(at 231.14 114.3 0)
-		(mirror y)
-		(unit 1)
-		(exclude_from_sim no)
-		(in_bom yes)
-		(on_board yes)
-		(dnp no)
-		(property "Reference" "J4"
-			(at 228.6 114.2999 0)
-			(effects
-				(font
-					(size 1.27 1.27)
-				)
-				(justify left)
-			)
-		)
-		(property "Value" "SSB"
-			(at 228.6 116.8399 0)
-			(effects
-				(font
-					(size 1.27 1.27)
-				)
-				(justify left)
-			)
-		)
-		(property "Footprint" "Connector_PinHeader_2.54mm:PinHeader_1x02_P2.54mm_Vertical"
-			(at 231.14 114.3 0)
-			(effects
-				(font
-					(size 1.27 1.27)
-				)
-				(hide yes)
-			)
-		)
-		(property "Datasheet" "~"
-			(at 231.14 114.3 0)
-			(effects
-				(font
-					(size 1.27 1.27)
-				)
-				(hide yes)
-			)
-		)
-		(property "Description" "Generic connector, single row, 01x02, script generated (kicad-library-utils/schlib/autogen/connector/)"
-			(at 231.14 114.3 0)
-			(effects
-				(font
-					(size 1.27 1.27)
-				)
-				(hide yes)
-			)
-		)
-		(pin "2"
-		)
-		(pin "1"
-		)
-		(instances
-			(project "Odb225GUM_JKK_TEST"
-				(path "/fd24851e-81c8-49e1-a423-2c617f6dbaa3"
-					(reference "J4")
-					(unit 1)
-				)
